File: Pressure Broom 2/Pressure Broom 2.kicad_sch (KiCad schematic)
At the start: 65 parts, among them J1 FTSH-105-01-F-DV-P-TR, J2 TYPE-C-31-M-12, Q1 FS8205, SW1 Power, U1 AP2127K-1.8, U2 MCP6004, U3 TCA9517D, U4 AP2127K-3.3, U5 ICM-20948, U6 DW01A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

Commit message: Documentation and Flexiforce datasheets
Other:
- note added: "PWM filter and buffer"
- note added: "Power via 3.7V LiPo, nRF5340 accepts 5V power. Boost circuit to boost 3.7V LiPo to 5V. Battery recharging at 1A from USB-C."
- note added: "Power: The nRF5340 module that I'm using (Laird 453-00052R) can accept a 5V power source but has internal 3V3 VDD even when powered from 5V. ADCs are used to read back the V_REF, V_BIAS, and pressure voltages which are shifted from 5Vs in the op amps to max 3V3 for the ADCs (can take max VDD + 0V3). The whole system will be powered from a 3V7 LiPo through a boost converter to 5V. Shouldn't take m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"
- note added: "This circuit intends to connect two pressure senssors (Tekscan Flexiforce A502) and an IMU to a bluetooth module. It's meant to measure pressure and frequency of motion when a curler sweeps (typically around oscillating 150-250 lbs @ a few Hz). The pressure sensors act as variable resistors from about 2M unloaded to 10k at 200 lbs. I've tested the MCP6004 circuit (their recommended integration ap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"
- note removed: "Power via 3.7V LiPo or USB-C. nRF5340 accepts 5V power. Buck boost circuit to boost 3.7V LiPo to 5V. Battery recharging at 1A."
Changed lines of the file:
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@@
 		)
 	)
-	(text "Power via 3.7V LiPo or USB-C.\nnRF5340 accepts 5V power.\nBuck boost circuit to boost 3.7V LiPo to 5V.\nBattery recharging at 1A."
+	(text "Power via 3.7V LiPo, nRF5340 accepts 5V power. Boost circuit to boost 3.7V LiPo to 5V.\nBattery recharging at 1A from USB-C."
 		(exclude_from_sim no)
 		(at 350.52 26.162 0)
@@
 				(size 1.27 1.27)
 				(thickness 0.1588)
+			)
+		)
+	)
+	(text "This circuit intends to connect two pressure senssors (Tekscan Flexiforce A502)\nand an IMU to a bluetooth module. It's meant to measure pressure and frequency\nof motion when a curler sweeps (typically around oscillating 150-250 lbs @ a \nfew Hz). \n\nThe pressure sensors act as variable resistors from about 2M unloaded to 10k \nat 200 lbs. I've tested the MCP6004 circuit (their recommended integration \napproach) with a breadboard and Arduino Nano supplying PWM V_REF and V_BIAS,\nthat all seemed to work fine. I'm using the PWM so that I can change the \nsensitivity range of the sensor after production if needed by varying the \nvalues.\n\nThe IMU is untested but very similar to the one we use on P-ONE, I2C with\na 1V8 level shift. It just needs to read at a couple hundred Hz to get a\nfrequency of motion and maybe a basic speed integration. Magnetic sensor\nis in there for orientation."
+		(exclude_from_sim no)
+		(at 72.39 129.54 0)
+		(effects
+			(font
+				(size 1.27 1.27)
 			)
 		)
@@
 		)
 	)
+	(text "PWM filter and buffer"
+		(exclude_from_sim no)
+		(at 43.434 26.162 0)
+		(effects
+			(font
+				(size 1.27 1.27)
+			)
+		)
+	)
 	(text "I2C levels are shifted from 3V3 (nRF5340) to\n1V8 (ICM-20948). Pull-up resistors are 10k and\nimplemented here. AD0 is selected low for ICM-20948."
 		(exclude_from_sim no)
@@
 			)
 		)
+	)
+	(text "Power:\n\nThe nRF5340 module that I'm using (Laird 453-00052R) can accept a 5V power source\nbut has internal 3V3 VDD even when powered from 5V. ADCs are used to read back the\nV_REF, V_BIAS, and pressure voltages which are shifted from 5Vs in the op amps to\nmax 3V3 for the ADCs (can take max VDD + 0V3). The whole system will be powered \nfrom a 3V7 LiPo through a boost converter to 5V. Shouldn't take more than 10s of\nmA, maybe lower. LDOs convert 5V to 3V3 and 1V8 for the I2C communications."
+		(exclude_from_sim no)
+		(at 234.696 176.784 0)
+		(effects
+			(font
+				(size 1.27 1.27)
+			)
+		)
